File: Hardware/IoT Controller/SkyKontrol-IotController.sch (EAGLE design)
At the start: 42 parts, among them IC1 NCP1117DT33G, J4 SBH11-PBPC-D05, K1 G5LE, SW1 SPST_TACT-EVQQ2, SW2 SPST_TACT-EVQQ2, T1 MMBT3904, T2 MMBT3904, T3 MMBT3904

Commit message: documentation add
Changed lines of the file:
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@@
 <?xml version="1.0" encoding="utf-8"?>
 <!DOCTYPE eagle SYSTEM "eagle.dtd">
-<eagle version="9.4.2">
+<eagle version="9.5.2">
 <drawing>
 <settings>
@@
 <part name="SW2" library="adafruit" deviceset="SPST_TACT" device="-EVQQ2"/>
 <part name="K1" library="relay" library_urn="urn:adsk.eagle:library:339" deviceset="G5LE" device="" package3d_urn="urn:adsk.eagle:package:24308/1"/>
-<part name="T2" library="transistor" library_urn="urn:adsk.eagle:library:402" deviceset="*-NPN-" device="SOT23-BEC" package3d_urn="urn:adsk.eagle:package:29919/2" technology="MMBT3904LT1" value="MMBT3904"/>
+<part name="T2" library="transistor" library_urn="urn:adsk.eagle:library:402" deviceset="*-NPN-" device="SOT23-BEC" package3d_urn="urn:adsk.eagle:package:28748/2" technology="MMBT3904LT1" value="MMBT3904"/>
 <part name="J1" library="SparkFun-Connectors" deviceset="CONN_03" device="-SCREW-5MM"/>
 <part name="J3" library="SparkFun-Connectors" deviceset="CONN_03" device="-SCREW-5MM"/>
@@
 <part name="C5" library="Panasonic-EEEFT_EEEH" deviceset="EEE-" device="-CASE-D8" technology="HA1E101XP" value="100UF"/>
 <part name="X1" library="adafruit" deviceset="ESP-12" device=""/>
-<part name="T1" library="transistor" library_urn="urn:adsk.eagle:library:402" deviceset="*-NPN-" device="SOT23-BEC" package3d_urn="urn:adsk.eagle:package:29919/2" technology="MMBT3904LT1" value="MMBT3904"/>
+<part name="T1" library="transistor" library_urn="urn:adsk.eagle:library:402" deviceset="*-NPN-" device="SOT23-BEC" package3d_urn="urn:adsk.eagle:package:28748/2" technology="MMBT3904LT1" value="MMBT3904"/>
 <part name="R5" library="adafruit" deviceset="R-US_" device="R0805" value="10k"/>
 <part name="R7" library="adafruit" deviceset="R-US_" device="R0805" value="2k2"/>
 <part name="R8" library="adafruit" deviceset="R-US_" device="R0805" value="2k2"/>
 <part name="J2" library="SparkFun-Connectors" deviceset="CONN_03" device="-SCREW-5MM"/>
-<part name="T3" library="transistor" library_urn="urn:adsk.eagle:library:402" deviceset="*-NPN-" device="SOT23-BEC" package3d_urn="urn:adsk.eagle:package:29919/2" technology="MMBT3904LT1" value="MMBT3904"/>
+<part name="T3" library="transistor" library_urn="urn:adsk.eagle:library:402" deviceset="*-NPN-" device="SOT23-BEC" package3d_urn="urn:adsk.eagle:package:28748/2" technology="MMBT3904LT1" value="MMBT3904"/>
 <part name="GND5" library="SparkFun-PowerSymbols" deviceset="GND" device=""/>
 <part name="R1" library="adafruit" deviceset="R-US_" device="R0805" value="2k2"/>
@@
 <part name="R15" library="adafruit" deviceset="R-US_" device="R0805" value="10k"/>
 <part name="R16" library="adafruit" deviceset="R-US_" device="R0805" value="10k"/>
+<part name="SUPPLY10" library="SparkFun-PowerSymbols" library_urn="urn:adsk.eagle:library:530" deviceset="3.3V" device=""/>
 </parts>
 <sheets>
@@
 <attribute name="NAME" x="112.8014" y="95.25" size="1.778" layer="95" rot="R90"/>
 <attribute name="VALUE" x="117.602" y="95.25" size="1.778" layer="96" rot="R90"/>
+</instance>
+<instance part="SUPPLY10" gate="G$1" x="109.22" y="111.76" smashed="yes">
+<attribute name="VALUE" x="109.22" y="114.554" size="1.778" layer="96" align="bottom-center"/>
 </instance>
 </instances>
@@
 <pinref part="R15" gate="G$1" pin="2"/>
 <wire x1="104.14" y1="104.14" x2="104.14" y2="106.68" width="0.1524" layer="91"/>
+<pinref part="R16" gate="G$1" pin="2"/>
 <wire x1="104.14" y1="106.68" x2="109.22" y2="106.68" width="0.1524" layer="91"/>
-<pinref part="R16" gate="G$1" pin="2"/>
 <wire x1="109.22" y1="106.68" x2="114.3" y2="106.68" width="0.1524" layer="91"/>
 <wire x1="114.3" y1="106.68" x2="114.3" y2="104.14" width="0.1524" layer="91"/>
-<wire x1="109.22" y1="106.68" x2="109.22" y2="111.76" width="0.1524" layer="91"/>
+<pinref part="SUPPLY10" gate="G$1" pin="3.3V"/>
+<wire x1="109.22" y1="111.76" x2="109.22" y2="106.68" width="0.1524" layer="91"/>
 <junction x="109.22" y="106.68"/>
-<junction x="109.22" y="111.76"/>
-<label x="106.68" y="114.3" size="1.778" layer="95"/>
-</segment>
-</net>
+</segment>
+</net>
