File: Hardware/IoT Controller/SkyKontrol-IotController.brd (EAGLE design)
At the start: 50 x 100 mm, 42 parts, among them IC1 NCP1117DT33G, J4 SBH11-PBPC-D05, K1 G5LE, SW1 SPST_TACT-EVQQ2, SW2 SPST_TACT-EVQQ2, T1 MMBT3904, T2 MMBT3904, T3 MMBT3904

Commit message: documentation add
Changed lines of the file:
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@@
 <?xml version="1.0" encoding="utf-8"?>
 <!DOCTYPE eagle SYSTEM "eagle.dtd">
-<eagle version="9.4.2">
+<eagle version="9.5.2">
 <drawing>
 <settings>
@@
 <attribute name="OC_FARNELL" value="unknown" x="25" y="25" size="1.778" layer="27" rot="R270" display="off"/>
 <attribute name="OC_NEWARK" value="unknown" x="25" y="25" size="1.778" layer="27" rot="R270" display="off"/>
+<attribute name="POPULARITY" value="13" x="25" y="25" size="1.778" layer="27" rot="R270" display="off"/>
 <attribute name="VALUE" x="17.38" y="15.475" size="1.778" layer="27" ratio="10"/>
 </element>
@@
 <element name="SW1" library="adafruit" package="EVQ-Q2" value="SPST_TACT-EVQQ2" x="9.5" y="46.5" smashed="yes" rot="R180"/>
 <element name="SW2" library="adafruit" package="EVQ-Q2" value="SPST_TACT-EVQQ2" x="21" y="46.5" smashed="yes"/>
-<element name="T2" library="transistor" library_urn="urn:adsk.eagle:library:402" package="SOT23-BEC" package3d_urn="urn:adsk.eagle:package:29919/2" value="MMBT3904" x="3.5" y="30.5" smashed="yes" rot="R180"/>
+<element name="T2" library="transistor" library_urn="urn:adsk.eagle:library:402" package="SOT23-BEC" package3d_urn="urn:adsk.eagle:package:28748/2" value="MMBT3904" x="3.5" y="30.5" smashed="yes" rot="R180">
+<attribute name="POPULARITY" value="0" x="3.5" y="30.5" size="1.778" layer="27" rot="R180" display="off"/>
+</element>
 <element name="C1" library="Panasonic-EEEFT_EEEH" package="CAPAE660X800N" value="100UF" x="43.5" y="80" smashed="yes" rot="R180">
 <attribute name="MPN" value="EEE-HA1E101XP" x="43.5" y="80" size="1.778" layer="27" rot="R180" display="off"/>
@@
 <attribute name="VALUE" x="25.5" y="69.5" size="1.4224" layer="27" font="vector" ratio="12" rot="R90" align="center"/>
 </element>
-<element name="T1" library="transistor" library_urn="urn:adsk.eagle:library:402" package="SOT23-BEC" package3d_urn="urn:adsk.eagle:package:29919/2" value="MMBT3904" x="3.5" y="36.5" smashed="yes" rot="R180"/>
+<element name="T1" library="transistor" library_urn="urn:adsk.eagle:library:402" package="SOT23-BEC" package3d_urn="urn:adsk.eagle:package:28748/2" value="MMBT3904" x="3.5" y="36.5" smashed="yes" rot="R180">
+<attribute name="POPULARITY" value="0" x="3.5" y="36.5" size="1.778" layer="27" rot="R180" display="off"/>
+</element>
 <element name="R5" library="adafruit" package="R0805" value="10k" x="8.5" y="35" smashed="yes"/>
 <element name="R7" library="adafruit" package="R0805" value="2k2" x="8.5" y="32" smashed="yes"/>
@@
 <attribute name="VALUE" x="20.929" y="93.905" size="0.6096" layer="27" font="vector" ratio="20"/>
 </element>
-<element name="T3" library="transistor" library_urn="urn:adsk.eagle:library:402" package="SOT23-BEC" package3d_urn="urn:adsk.eagle:package:29919/2" value="MMBT3904" x="3.5" y="87" smashed="yes"/>
+<element name="T3" library="transistor" library_urn="urn:adsk.eagle:library:402" package="SOT23-BEC" package3d_urn="urn:adsk.eagle:package:28748/2" value="MMBT3904" x="3.5" y="87" smashed="yes">
+<attribute name="POPULARITY" value="0" x="3.5" y="87" size="1.778" layer="27" display="off"/>
+</element>
 <element name="R1" library="adafruit" package="R0805" value="2k2" x="3" y="82" smashed="yes" rot="R270"/>
 <element name="J4" library="con-sullins" package="SBH11-PBPC-D05" value="SBH11-PBPC-D05" x="42.5" y="25" smashed="yes" rot="R90"/>

Commit message: update
Other:
- board text added: "2brobots"
- board text added: "R2.2"
- board text removed: "Desarrollado por:"
- board text removed: "R2.1"
