File: Hardware/Datalogger/SkyKontrol-datalogger.sch (EAGLE design)
At the start: 23 parts, among them J4 SBH11-PBPC-D05, T1 MMBT3904, T2 MMBT3904, U1 PIC12F1822-E/SN

Commit message: update
Parts:
- removed C4: 100UF, Panasonic-EEEFT_EEEH:EEE-HA1E101XP-CASE-D8
- removed DS1: NHD-C0220BIZ-FSW-FBW-3V3M, NHD-C0220BIZ-FSW-FBW-3V3M:NHD-C0220BIZ-FSW-FBW-3V3M
- removed LS1: CMI-9651S-SMT, CMI-9651S-SMT:CMI-9651S-SMT
- removed R4, R5: 2K2, adafruit:R-US_R0805
- removed R6: 10k, adafruit:R-US_R0805
- removed T1, T2: MMBT3904, transistor:MMBT3904LT1-NPN-SOT23-BEC
- removed U$2: ICSP_POGO, ICSP_POGO:ICSP_POGO
- removed U1: PIC12F1822-E/SN, Microchip-PIC12F1822-E_SN:PIC12F1822-E/SN
- added B2: CR1220, microbuilder:BATTERYCR1220_SMT
- added IC3: RTC_PCF8523T, microbuilder:RTC_PCF8523T
- added Q1: 32.768, microbuilder:CRYSTAL8.0X3.8
- added U2: MB85RC256VPF-G-JNERE2, microbuilder:FRAM_SOIC8_I2C
- C1: value 1uF -> 100UF; device adafruit:C-USC0603K -> Panasonic-EEEFT_EEEH:EEE-HA1E101XP-CASE-D8
- C2: value 1uF -> 100nF
- C3: value 100nF -> 10uF; device adafruit:C-USC0603K -> adafruit:C-USC0805K
- JP1: value JUMPER-SMT_3_1-NC_PASTE_SILK -> JUMPER-SMT_2_NO_SILK; device SparkFun-Jumpers:JUMPER-SMT_3_1-NC_PASTE_SILK -> SparkFun-Jumpers:JUMPER-SMT_2_NO_SILK
- JP4: value (none) -> JUMPER-SMT_2_NO_SILK; device adafruit:PINHD-1X3CB -> SparkFun-Jumpers:JUMPER-SMT_2_NO_SILK
- R1: value 10ohm -> 10K
- R3: value 10K -> 1k
Connections:
- removed net DAT: R4.1, U$2.DAT, U1.RA0/ICSPDAT
- removed net N$10: LS1.N, T1.C
- removed net N$12: R4.2, T1.B
- removed net N$17: DS1.K, T2.C
- removed net N$19: R5.2, T2.B
- removed net PWM: R5.1, U1.RA5
- removed net RA3: JP3.1, U$2.RST, U1.!MCLR!/VPP/RA3
- removed net RSTS: DS1.RST, JP1.2, JP3.2
- removed net SEN: JP4.2, R6.1, U1.RA4
- new net N$14: IC3.XI, Q1.1
- new net N$15: IC3.XO, Q1.2
- new net VBAT1: B2.+, IC3.VBAT
- net 12V: no longer LS1.P
- net 3.3V: now also C1.1, C2.1, JP2.1, JP3.1, JP4.2, R3.2, U2.VCC; no longer C3.1, C4.1, DS1.VDD, JP2.2, JP4.1, R1.2, U$2.VDD, U1.VDD
- net GND: now also B2.-, C1.2, IC3.VSS, U2.GND; no longer C4.2, DS1.VSS, JP4.3, R6.2, T1.E, T2.E, U$2.GND, U1.VSS
- net N$1: now also JP1.2, U2.A0; no longer C2.1, DS1.VOUT
- net N$2: now also JP2.2, U2.A1; no longer C1.2, DS1.C1-
- net N$3: now also C3.1, IC3.VDD, R3.1; no longer C1.1, DS1.C1+
- net N$4: now also JP3.2, U2.A2; no longer DS1.A, R1.1
- net N$8: now also JP4.1, R1.2; no longer JP2.1, R3.2
- net RST: no longer JP1.3
- net SCL: now also IC3.SCL, R2.1, U2.SCL; no longer DS1.SCL, R3.1, U$2.CLK, U1.RA1/ICSPCLK
- net SDA: now also IC3.SDA, R1.1, U2.SDA; no longer DS1.SDA, R2.1, U1.RA2
Other:
- moved on the sheet: C2, C3, J4, JP2, JP3, R1, R2, R3
