File: Hardware/Power Meter/SkyKontrol-powerMeter.brd (EAGLE design)
At the start: 60 x 50 mm, 25 parts, among them J4 SBH11-PBPC-D05, U1 PIC12F1822-E/SN

Commit message: update
Routing:
- net RA3: track 95.0 -> 96.3 mm
Changed lines of the file:
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@@
 <wire x1="41.9" y1="25" x2="40.0378" y2="23.1378" width="0.6096" layer="1"/>
 <wire x1="3.95" y1="14" x2="3.95" y2="11.05" width="0.6096" layer="1"/>
-<wire x1="7.5" y1="7.5" x2="25" y2="7.5" width="0.6096" layer="1"/>
-<wire x1="35" y1="5.5" x2="37.5" y2="3" width="0.6096" layer="1"/>
 <wire x1="37.5" y1="3" x2="48.5" y2="3" width="0.6096" layer="1"/>
 <wire x1="48.5" y1="3" x2="50.5" y2="5" width="0.6096" layer="1"/>
@@
 <wire x1="55.5" y1="14" x2="55.5" y2="21" width="0.6096" layer="1"/>
 <wire x1="3.95" y1="11.05" x2="7.5" y2="7.5" width="0.6096" layer="1"/>
-<wire x1="25" y1="7.5" x2="27" y2="5.5" width="0.6096" layer="1"/>
-<wire x1="27" y1="5.5" x2="35" y2="5.5" width="0.6096" layer="1"/>
 <wire x1="53.3622" y1="23.1378" x2="55.5" y2="21" width="0.6096" layer="1"/>
 <wire x1="40.0378" y1="23.1378" x2="53.3622" y2="23.1378" width="0.6096" layer="1"/>
+<wire x1="36" y1="1.5" x2="37.5" y2="3" width="0.6096" layer="1"/>
+<wire x1="7.5" y1="7.5" x2="19.5" y2="7.5" width="0.6096" layer="1"/>
+<wire x1="19.5" y1="7.5" x2="25.5" y2="1.5" width="0.6096" layer="1"/>
+<wire x1="25.5" y1="1.5" x2="36" y2="1.5" width="0.6096" layer="1"/>
 </signal>
 <signal name="ADC2">
