File: Hardware/Smart Display/SkyKontrol-smartDisplay.brd (EAGLE design)
At the start: 94 x 40 mm, 23 parts, among them J4 SBH11-PBPC-D05, T1 MMBT3904, T2 MMBT3904, U1 PIC12F1822-E/SN

Commit message: documentation add
Changed lines of the file:
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@@
 <setting verticaltext="up"/>
 </settings>
-<grid distance="1" unitdist="mm" unit="mm" style="lines" multiple="1" display="yes" altdistance="5" altunitdist="mil" altunit="mil"/>
+<grid distance="0.1" unitdist="mm" unit="mm" style="lines" multiple="1" display="yes" altdistance="5" altunitdist="mil" altunit="mil"/>
 <layers>
 <layer number="1" name="Top" color="4" fill="1" visible="yes" active="yes"/>
@@
 <element name="R6" library="adafruit" package="R0805" value="10k" x="70.7" y="22.9" smashed="yes" rot="MR270"/>
 <element name="R5" library="adafruit" package="R0805" value="2K2" x="31.8" y="32" smashed="yes" rot="MR0"/>
-<element name="T2" library="transistor" library_urn="urn:adsk.eagle:library:402" package="SOT23-BEC" package3d_urn="urn:adsk.eagle:package:29919/2" value="MMBT3904" x="26.1" y="31.1" smashed="yes" rot="MR270"/>
+<element name="T2" library="transistor" library_urn="urn:adsk.eagle:library:402" package="SOT23-BEC" package3d_urn="urn:adsk.eagle:package:28748/2" value="MMBT3904" x="26.1" y="31.1" smashed="yes" rot="MR270">
+<attribute name="POPULARITY" value="0" x="26.1" y="31.1" size="1.778" layer="28" rot="MR270" display="off"/>
+</element>
 <element name="U$2" library="ICSP_POGO" package="ICSP_POGO" value="ICSP_POGO" x="52.9" y="22.1" smashed="yes" rot="MR0">
 <attribute name="PIC" value="" x="129.9" y="-27.9" size="1.778" layer="28" rot="MR0" display="off"/>
@@
 </element>
 <element name="R4" library="adafruit" package="R0805" value="2K2" x="79.5" y="26.5" smashed="yes" rot="MR90"/>
-<element name="T1" library="transistor" library_urn="urn:adsk.eagle:library:402" package="SOT23-BEC" package3d_urn="urn:adsk.eagle:package:29919/2" value="MMBT3904" x="68" y="36.4" smashed="yes" rot="MR270"/>
+<element name="T1" library="transistor" library_urn="urn:adsk.eagle:library:402" package="SOT23-BEC" package3d_urn="urn:adsk.eagle:package:28748/2" value="MMBT3904" x="68" y="36.4" smashed="yes" rot="MR270">
+<attribute name="POPULARITY" value="0" x="68" y="36.4" size="1.778" layer="28" rot="MR270" display="off"/>
+</element>
 <element name="LS1" library="CMI-9651S-SMT" package="CUI_CMI-9651S-SMT" value="CMI-9651S-SMT" x="19.3" y="22.4" smashed="yes" rot="MR270">
 <attribute name="MANUFACTURER" value="CUI INC" x="19.3" y="22.4" size="1.778" layer="28" rot="MR270" display="off"/>
@@
 <wire x1="90.27" y1="14.92" x2="90.27" y2="14.07" width="0.6096" layer="16"/>
 <wire x1="70.6" y1="12.8" x2="68.8" y2="14.6" width="0.6096" layer="16"/>
-<via x="68.8" y="14.6" extent="1-16" drill="0.35"/>
+<via x="68.8" y="14.6" extent="1-16" drill="0.4"/>
 <wire x1="68.8" y1="14.6" x2="30.1" y2="14.6" width="0.6096" layer="1"/>
 <wire x1="27.2" y1="17.5" x2="25.7" y2="17.5" width="0.6096" layer="1"/>
-<via x="25.7" y="17.5" extent="1-16" drill="0.35"/>
+<via x="25.7" y="17.5" extent="1-16" drill="0.4"/>
 <wire x1="25.7" y1="17.5" x2="19.5" y2="17.5" width="0.6096" layer="16"/>
 <wire x1="19.5" y1="17.5" x2="19.4" y2="17.4" width="0.6096" layer="16"/>
@@
 <contactref element="JP4" pad="3"/>
 <contactref element="R6" pad="2"/>
+<via x="74" y="15" extent="1-16" drill="0.4"/>
 </signal>
 <signal name="RST">
@@
 <contactref element="U1" pad="6"/>
 <contactref element="U$2" pad="P$5"/>
-<wire x1="75.635" y1="23.6378" x2="75.635" y2="18.7" width="0.6096" layer="16"/>
-<via x="75.635" y="18.7" extent="1-16" drill="0.35"/>
-<wire x1="75.635" y1="18.7" x2="75.635" y2="11.4" width="0.6096" layer="1"/>
+<wire x1="75.635" y1="23.6378" x2="75.635" y2="18.75" width="0.6096" layer="16"/>
+<via x="75.635" y="18.75" extent="1-16" drill="0.4"/>
+<wire x1="75.635" y1="18.75" x2="75.635" y2="11.4" width="0.6096" layer="1"/>
 <wire x1="51.625" y1="24" x2="47.1" y2="24" width="0.6096" layer="16"/>
-<via x="47.1" y="24" extent="1-16" drill="0.35"/>
+<via x="47.1" y="24" extent="1-16" drill="0.4"/>
 <wire x1="47.1" y1="24" x2="47.1" y2="21" width="0.6096" layer="1"/>
 <wire x1="50.2" y1="17.9" x2="56.3" y2="17.9" width="0.6096" layer="1"/>
-<via x="56.3" y="17.9" extent="1-16" drill="0.35"/>
+<via x="56.3" y="17.9" extent="1-16" drill="0.4"/>
 <wire x1="56.3" y1="17.9" x2="56.3" y2="13.2" width="0.6096" layer="16"/>
 <wire x1="56.3" y1="13.2" x2="56" y2="12.9" width="0.6096" layer="16"/>
@@
 <wire x1="72" y1="14" x2="72" y2="18" width="0.6096" layer="1"/>
 <wire x1="72" y1="18" x2="74" y2="20" width="0.6096" layer="1"/>
-<wire x1="74" y1="20" x2="76.9" y2="20" width="0.6096" layer="1"/>
-<wire x1="76.9" y1="20" x2="87.73" y2="20" width="0.6096" layer="1"/>
+<wire x1="74" y1="20" x2="77" y2="20" width="0.6096" layer="1"/>
+<wire x1="77" y1="20" x2="87.73" y2="20" width="0.6096" layer="1"/>
 <wire x1="70" y1="12" x2="54" y2="12" width="0.6096" layer="1"/>
 <wire x1="54" y1="12" x2="52.058" y2="10.058" width="0.6096" layer="1"/>
@@
 <wire x1="52.058" y1="12.942" x2="52.058" y2="7.35" width="0.6096" layer="16"/>
 <contactref element="U1" pad="5"/>
-<wire x1="76.905" y1="23.6378" x2="76.905" y2="18.7" width="0.6096" layer="16"/>
-<wire x1="76.905" y1="18.7" x2="76.9" y2="18.7" width="0.6096" layer="16"/>
-<via x="76.9" y="18.7" extent="1-16" drill="0.35"/>
-<wire x1="76.9" y1="18.7" x2="76.9" y2="20" width="0.6096" layer="1"/>
+<via x="77" y="18.75" extent="1-16" drill="0.4"/>
+<wire x1="77" y1="18.75" x2="77" y2="20" width="0.6096" layer="1"/>
+<wire x1="76.905" y1="23.6378" x2="76.905" y2="21.695" width="0.6096" layer="16"/>
+<wire x1="77" y1="18.75" x2="77" y2="21.6" width="0.6096" layer="16"/>
+<wire x1="77" y1="21.6" x2="76.905" y2="21.695" width="0.6096" layer="16"/>
 </signal>
 <signal name="3.3V">
@@
 <wire x1="48.125" y1="4.375" x2="48.1" y2="4.4" width="0.6096" layer="16"/>
 <wire x1="48.1" y1="4.4" x2="30.4" y2="4.4" width="0.6096" layer="16"/>
-<wire x1="52.89" y1="22.1" x2="52.89" y2="20.11" width="0.6096" layer="16"/>
+<wire x1="52.9" y1="22.1" x2="52.89" y2="20.11" width="0.6096" layer="16"/>
 <wire x1="52.89" y1="20.11" x2="53" y2="20" width="0.6096" layer="16"/>
 <wire x1="68.5" y1="25.6" x2="68.5" y2="17.46" width="0.6096" layer="16"/>
@@
 <wire x1="60.0064" y1="22.1" x2="62" y2="22.1" width="0.6096" layer="16"/>
 <wire x1="62" y1="22.1" x2="62.3" y2="21.8" width="0.6096" layer="16"/>
-<via x="62.3" y="21.8" extent="1-16" drill="0.35"/>
+<via x="62.3" y="21.8" extent="1-16" drill="0.4"/>
 <wire x1="62.3" y1="21.8" x2="64.5" y2="19.6" width="0.6096" layer="1"/>
 <wire x1="64.5" y1="19.6" x2="64.5" y2="16.6" width="0.6096" layer="1"/>
-<via x="64.5" y="16.6" extent="1-16" drill="0.35"/>
+<via x="64.5" y="16.6" extent="1-16" drill="0.4"/>
 <wire x1="64.5" y1="16.6" x2="64.5" y2="7.475" width="0.6096" layer="16"/>
 <wire x1="64.5" y1="7.475" x2="64.6" y2="7.375" width="0.6096" layer="16"/>
@@
 <wire x1="76.905" y1="28.3622" x2="76.905" y2="30.695" width="0.6096" layer="16"/>
 <wire x1="76.905" y1="30.695" x2="76.9" y2="30.7" width="0.6096" layer="16"/>
-<via x="76.9" y="30.7" extent="1-16" drill="0.35"/>
+<via x="76.9" y="30.7" extent="1-16" drill="0.4"/>
 <wire x1="76.9" y1="30.7" x2="58.9" y2="30.7" width="0.6096" layer="1"/>
 <wire x1="57.7" y1="29.5" x2="57.7" y2="24.3" width="0.6096" layer="1"/>
-<via x="57.7" y="24.3" extent="1-16" drill="0.35"/>
+<via x="57.7" y="24.3" extent="1-16" drill="0.4"/>
 <wire x1="57.7" y1="24.3" x2="57.7" y2="22.1" width="0.6096" layer="16"/>
 <wire x1="58.9" y1="30.7" x2="57.7" y2="29.5" width="0.6096" layer="1"/>
@@
 <wire x1="54.7" y1="26.1" x2="61" y2="26.1" width="0.6096" layer="16"/>
 <wire x1="61" y1="26.1" x2="65.9" y2="21.2" width="0.6096" layer="16"/>
-<via x="65.9" y="21.2" extent="1-16" drill="0.35"/>
+<via x="65.9" y="21.2" extent="1-16" drill="0.4"/>
 <wire x1="65.9" y1="21.2" x2="73.4" y2="21.2" width="0.6096" layer="1"/>
 <wire x1="73.4" y1="21.2" x2="73.5" y2="21.3" width="0.6096" layer="1"/>
-<via x="73.5" y="21.3" extent="1-16" drill="0.35"/>
+<via x="73.5" y="21.3" extent="1-16" drill="0.4"/>
 <wire x1="73.5" y1="21.3" x2="74.365" y2="22.165" width="0.6096" layer="16"/>
 <wire x1="74.365" y1="22.165" x2="74.365" y2="23.6378" width="0.6096" layer="16"/>
@@
 <contactref element="R6" pad="1"/>
 <wire x1="70.7" y1="23.9" x2="70.7" y2="25.1" width="0.6096" layer="16"/>
-<wire x1="72" y1="26.4" x2="74.9" y2="26.4" width="0.6096" layer="16"/>
-<wire x1="74.9" y1="26.4" x2="75.635" y2="27.135" width="0.6096" layer="16"/>
-<wire x1="75.635" y1="27.135" x2="75.635" y2="28.3622" width="0.6096" layer="16"/>
+<wire x1="72" y1="26.4" x2="75.1" y2="26.4" width="0.6096" layer="16"/>
+<wire x1="75.1" y1="26.4" x2="75.635" y2="26.935" width="0.6096" layer="16"/>
+<wire x1="75.635" y1="26.935" x2="75.635" y2="28.3622" width="0.6096" layer="16"/>
 <wire x1="70.7" y1="25.1" x2="72" y2="26.4" width="0.6096" layer="16"/>
 <contactref element="JP4" pad="2"/>
 <wire x1="75.635" y1="28.3622" x2="75.635" y2="32.565" width="0.6096" layer="16"/>
 <wire x1="74.3" y1="33.9" x2="42.2" y2="33.9" width="0.6096" layer="16"/>
-<via x="42.2" y="33.9" extent="1-16" drill="0.35"/>
+<via x="42.2" y="33.9" extent="1-16" drill="0.4"/>
 <wire x1="42.2" y1="33.9" x2="37.8" y2="29.5" width="0.6096" layer="1"/>
 <wire x1="37.8" y1="29.5" x2="32.2" y2="29.5" width="0.6096" layer="1"/>
@@
 <wire x1="75.635" y1="32.565" x2="74.3" y2="33.9" width="0.6096" layer="16"/>
 <wire x1="25.2" y1="21.7" x2="12.8" y2="21.7" width="0.6096" layer="1"/>
-<via x="12.8" y="21.7" extent="1-16" drill="0.35"/>
+<via x="12.8" y="21.7" extent="1-16" drill="0.4"/>
 <wire x1="12.8" y1="21.7" x2="6.6" y2="21.7" width="0.6096" layer="16"/>
 <wire x1="4.9" y1="20" x2="2" y2="20" width="0.6096" layer="16"/>

Commit message: update
Parts:
- turned LS1 to 90 degrees
Changed lines of the file:
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@@
 <attribute name="POPULARITY" value="0" x="68" y="36.4" size="1.778" layer="28" rot="MR270" display="off"/>
 </element>
-<element name="LS1" library="CMI-9651S-SMT" package="CUI_CMI-9651S-SMT" value="CMI-9651S-SMT" x="19.3" y="22.4" smashed="yes" rot="MR270">
-<attribute name="MANUFACTURER" value="CUI INC" x="19.3" y="22.4" size="1.778" layer="28" rot="MR270" display="off"/>
-<attribute name="PARTREV" value="1.0" x="19.3" y="22.4" size="1.778" layer="28" rot="MR270" display="off"/>
-<attribute name="STANDARD" value="Manufacturer recommendations" x="19.3" y="22.4" size="1.778" layer="28" rot="MR270" display="off"/>
+<element name="LS1" library="CMI-9651S-SMT" package="CUI_CMI-9651S-SMT" value="CMI-9651S-SMT" x="19.3" y="22.4" smashed="yes" rot="MR90">
+<attribute name="MANUFACTURER" value="CUI INC" x="19.3" y="22.4" size="1.778" layer="28" rot="MR90" display="off"/>
+<attribute name="PARTREV" value="1.0" x="19.3" y="22.4" size="1.778" layer="28" rot="MR90" display="off"/>
+<attribute name="STANDARD" value="Manufacturer recommendations" x="19.3" y="22.4" size="1.778" layer="28" rot="MR90" display="off"/>
 </element>
 <element name="JP3" library="SparkFun-Jumpers" library_urn="urn:adsk.eagle:library:528" package="SMT-JUMPER_2_NO_SILK" package3d_urn="urn:adsk.eagle:package:39279/1" value="JUMPER-SMT_2_NO_SILK" x="59.6" y="22.1" smashed="yes" rot="MR180"/>
