File: Hardware/PowerMeter/SkyKontrol-powerMeter.brd (EAGLE design)
At the start: 60 x 50 mm, 25 parts, among them J4 SBH11-PBPC-D05, U1 PIC12F1822-E/SN

Commit message: BOM and corrections
Parts:
- R3: value 1k -> 120
- U1: value PIC12F1822-E/SN -> PIC12F1840-I/SN; device Microchip-PIC12F1822-E_SN:SOIC127P600X175-8N -> Microchip-PIC12F1840-I_SN:SOIC127P600X175-8N
Changed lines of the file:
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@@
 <element name="R2" library="adafruit" package="R0805" value="10K" x="21" y="27" smashed="yes" rot="R180"/>
 <element name="JP2" library="SparkFun-Jumpers" library_urn="urn:adsk.eagle:library:528" package="SMT-JUMPER_2_NO_SILK" package3d_urn="urn:adsk.eagle:package:39279/1" value="JUMPER-SMT_2_NO_SILK" x="17" y="28.5" smashed="yes" rot="R180"/>
-<element name="R3" library="adafruit" package="R0805" value="1k" x="16.5" y="14.5" smashed="yes" rot="R180"/>
+<element name="R3" library="adafruit" package="R0805" value="120" x="16.5" y="14.5" smashed="yes" rot="R180"/>
 <element name="U$2" library="ICSP_POGO" package="ICSP_POGO" value="ICSP_POGO" x="6.5" y="14" smashed="yes">
 <attribute name="PIC" value="" x="-70.5" y="-36" size="1.778" layer="27" display="off"/>
@@
 <attribute name="SMT" value="" x="-70.5" y="-36" size="1.778" layer="27" display="off"/>
 </element>
-<element name="U1" library="Microchip-PIC12F1822-E_SN" package="SOIC127P600X175-8N" value="PIC12F1822-E/SN" x="35" y="25.5" smashed="yes" rot="R90">
-<attribute name="MPN" value="PIC12F1822-E/SN" x="118" y="-48.5" size="1.778" layer="27" rot="R90" display="off"/>
-<attribute name="OC_FARNELL" value="2315760" x="118" y="-48.5" size="1.778" layer="27" rot="R90" display="off"/>
-<attribute name="OC_NEWARK" value="53R0195" x="118" y="-48.5" size="1.778" layer="27" rot="R90" display="off"/>
+<element name="U1" library="Microchip-PIC12F1840-I_SN" package="SOIC127P600X175-8N" value="PIC12F1840-I/SN" x="35" y="25.5" smashed="yes" rot="R90">
+<attribute name="MPN" value="PIC12F1840-I/SN" x="118" y="-48.5" size="1.778" layer="27" rot="R90" display="off"/>
+<attribute name="OC_FARNELL" value="1971859" x="118" y="-48.5" size="1.778" layer="27" rot="R90" display="off"/>
+<attribute name="OC_NEWARK" value="13T4707" x="118" y="-48.5" size="1.778" layer="27" rot="R90" display="off"/>
 <attribute name="PACKAGE" value="SOIC-8" x="118" y="-48.5" size="1.778" layer="27" rot="R90" display="off"/>
 <attribute name="SUPPLIER" value="Microchip" x="118" y="-48.5" size="1.778" layer="27" rot="R90" display="off"/>
