File: Hardware/PowerMeter/SkyKontrol-powerMeter.sch (EAGLE design)
At the start: 25 parts, among them J4 SBH11-PBPC-D05, U1 PIC12F1822-E/SN

Commit message: BOM and corrections
Parts:
- R3: value 1k -> 120
- U1: value PIC12F1822-E/SN -> PIC12F1840-I/SN; device Microchip-PIC12F1822-E_SN:PIC12F1822-E/SN -> Microchip-PIC12F1840-I_SN:PIC12F1840-I/SN
Changed lines of the file:
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@@
 <part name="R2" library="adafruit" deviceset="R-US_" device="R0805" value="10K"/>
 <part name="JP2" library="SparkFun-Jumpers" library_urn="urn:adsk.eagle:library:528" deviceset="JUMPER-SMT_2_NO" device="_SILK" package3d_urn="urn:adsk.eagle:package:39279/1"/>
-<part name="R3" library="adafruit" deviceset="R-US_" device="R0805" value="1k"/>
+<part name="R3" library="adafruit" deviceset="R-US_" device="R0805" value="120"/>
 <part name="U$2" library="ICSP_POGO" deviceset="ICSP_POGO" device=""/>
-<part name="U1" library="Microchip-PIC12F1822-E_SN" deviceset="PIC12F1822-E/SN" device=""/>
+<part name="U1" library="Microchip-PIC12F1840-I_SN" deviceset="PIC12F1840-I/SN" device=""/>
 <part name="GND3" library="SparkFun-PowerSymbols" deviceset="GND" device=""/>
 <part name="GND7" library="SparkFun-PowerSymbols" deviceset="GND" device=""/>
