File: Hardware/USB Terminal/usbTerminal.brd (EAGLE design)
At the start: 50 x 36 mm, 30 parts, among them IC1 MCP2221A-I_SL, J4 SBH11-PBPC-D05

Commit message: pcb corrected
Parts:
- removed JP8: JUMPER-SMT_2_NO_SILK, SparkFun-Jumpers:SMT-JUMPER_2_NO_SILK
- added S1: (no value), SparkFun-Switches:SWITCH_SPST_SMD_A
- moved U$3 2.50 mm to (38.0, 31.5)
Connections:
- net 3.3V: now also LED1.C, LED2.C, LED3.C, LED4.C, S1.2; no longer JP8.1
- net GND: now also S1.GND1, S1.GND2, S1.GND3, S1.GND4; no longer LED1.C, LED2.C, LED3.C, LED4.C
- net N$22: now also S1.1; no longer JP8.2
Routing:
- net 3.3V: track 74.9 -> 106.4 mm, vias 1 -> 5
- net N$22: track 8.82 -> 9.44 mm
Other:
- board text added: "R1.1"
- board text added: "RX"
- board text added: "TX"
- board text removed: "R1.0"

Commit message: LED polarity marks fix
Parts:
- turned LED1 to 180 degrees
- turned LED2 to 180 degrees
- turned LED3 to 180 degrees
- turned LED4 to 180 degrees
Connections:
- net 3.3V: now also LED1.A, LED2.A, LED3.A, LED4.A; no longer LED1.C, LED2.C, LED3.C, LED4.C
- net N$12: now also LED1.C, R3.1; no longer LED2.A, R4.1
- net N$13: now also LED2.C, R4.1; no longer LED1.A, R3.1
- net N$14: now also LED3.C; no longer LED3.A
- net N$15: now also LED4.C; no longer LED4.A
Changed lines of the file:
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@@
 <drawing>
 <settings>
-<setting alwaysvectorfont="no"/>
+<setting alwaysvectorfont="yes"/>
 <setting verticaltext="up"/>
 </settings>
@@
 <element name="JP7" library="SparkFun-Jumpers" library_urn="urn:adsk.eagle:library:528" package="SMT-JUMPER_2_NO_SILK" package3d_urn="urn:adsk.eagle:package:39279/1" value="JUMPER-SMT_2_NO_SILK" x="15" y="26" smashed="yes" rot="R270"/>
 <element name="R3" library="adafruit" package="R0805" value="330" x="26" y="3.5" smashed="yes" rot="R90"/>
-<element name="LED1" library="adafruit" package="CHIPLED_1206" value="Yellow (Rx)" x="24" y="3.5" smashed="yes"/>
+<element name="LED1" library="adafruit" package="CHIPLED_1206" value="Yellow (Rx)" x="24" y="3.5" smashed="yes" rot="R180"/>
 <element name="R4" library="adafruit" package="R0805" value="330" x="32" y="3.5" smashed="yes" rot="R90"/>
-<element name="LED2" library="adafruit" package="CHIPLED_1206" value="Yellow (Tx)" x="30" y="3.5" smashed="yes"/>
+<element name="LED2" library="adafruit" package="CHIPLED_1206" value="Yellow (Tx)" x="30" y="3.5" smashed="yes" rot="R180"/>
 <element name="R5" library="adafruit" package="R0805" value="330" x="38" y="3.5" smashed="yes" rot="R90"/>
-<element name="LED3" library="adafruit" package="CHIPLED_1206" value="Green (USB)" x="36" y="3.5" smashed="yes"/>
+<element name="LED3" library="adafruit" package="CHIPLED_1206" value="Green (USB)" x="36" y="3.5" smashed="yes" rot="R180"/>
 <element name="R6" library="adafruit" package="R0805" value="330" x="20" y="3.5" smashed="yes" rot="R90"/>
-<element name="LED4" library="adafruit" package="CHIPLED_1206" value="Red (I2C)" x="18" y="3.5" smashed="yes"/>
+<element name="LED4" library="adafruit" package="CHIPLED_1206" value="Red (I2C)" x="18" y="3.5" smashed="yes" rot="R180"/>
 <element name="U$2" library="MCP1700T-3302E" package="SOT95P237X112-3N" value="MCP1700T-3302E/TT" x="8.5" y="24" smashed="yes" rot="R90">
 <attribute name="MPN" value="MCP1700T-3302E/TT" x="8.5" y="24" size="1.778" layer="27" rot="R90" display="off"/>
@@
 <wire x1="34" y1="25" x2="31" y2="28" width="0.3048" layer="1"/>
 <wire x1="31" y1="28" x2="23" y2="28" width="0.3048" layer="1"/>
-<contactref element="LED3" pad="C"/>
-<contactref element="LED4" pad="C"/>
-<contactref element="LED1" pad="C"/>
-<contactref element="LED2" pad="C"/>
 <wire x1="14" y1="4.5" x2="16" y2="4.5" width="0.3048" layer="1"/>
-<wire x1="16.75" y1="5.25" x2="18" y2="5.25" width="0.3048" layer="1"/>
 <wire x1="16" y1="4.5" x2="16.75" y2="5.25" width="0.3048" layer="1"/>
 <wire x1="16" y1="4.5" x2="16" y2="6.5" width="0.3048" layer="1"/>
@@
 <wire x1="28" y1="5.5" x2="34" y2="5.5" width="0.3048" layer="16"/>
 <wire x1="19.5" y1="6.5" x2="20.5" y2="5.5" width="0.3048" layer="16"/>
-<wire x1="36" y1="5.25" x2="34.25" y2="5.25" width="0.3048" layer="1"/>
-<wire x1="34.25" y1="5.25" x2="34" y2="5.5" width="0.3048" layer="1"/>
+<wire x1="34" y1="5.5" x2="34.25" y2="5.25" width="0.3048" layer="1"/>
 <via x="34" y="5.5" extent="1-16" drill="0.35"/>
-<wire x1="24" y1="5.25" x2="22.25" y2="5.25" width="0.3048" layer="1"/>
-<wire x1="22.25" y1="5.25" x2="22" y2="5.5" width="0.3048" layer="1"/>
+<wire x1="22" y1="5.5" x2="22.25" y2="5.25" width="0.3048" layer="1"/>
 <via x="22" y="5.5" extent="1-16" drill="0.35"/>
-<wire x1="30" y1="5.25" x2="28.25" y2="5.25" width="0.3048" layer="1"/>
-<wire x1="28.25" y1="5.25" x2="28" y2="5.5" width="0.3048" layer="1"/>
+<wire x1="28" y1="5.5" x2="28.25" y2="5.25" width="0.3048" layer="1"/>
 <via x="28" y="5.5" extent="1-16" drill="0.35"/>
 <contactref element="S1" pad="2"/>
@@
 <wire x1="14.5" y1="30" x2="19" y2="30" width="0.3048" layer="1"/>
 <wire x1="19" y1="30" x2="21.5" y2="32.5" width="0.3048" layer="1"/>
+<contactref element="LED1" pad="A"/>
+<contactref element="LED2" pad="A"/>
+<contactref element="LED3" pad="A"/>
+<contactref element="LED4" pad="A"/>
+<wire x1="16.75" y1="5.25" x2="18" y2="5.25" width="0.3048" layer="1"/>
+<wire x1="22.25" y1="5.25" x2="24" y2="5.25" width="0.3048" layer="1"/>
+<wire x1="28.25" y1="5.25" x2="30" y2="5.25" width="0.3048" layer="1"/>
+<wire x1="34.25" y1="5.25" x2="36" y2="5.25" width="0.3048" layer="1"/>
 </signal>
 <signal name="N$3" airwireshidden="yes">
@@
 <wire x1="16.46" y1="20.54" x2="15" y2="22" width="0.3048" layer="1"/>
 <wire x1="15" y1="22" x2="15" y2="25.5936" width="0.3048" layer="1"/>
-</signal>
-<signal name="N$13">
-<contactref element="LED1" pad="A"/>
-<contactref element="R3" pad="1"/>
-<wire x1="24" y1="1.75" x2="25.75" y2="1.75" width="0.3048" layer="1"/>
-<wire x1="25.75" y1="1.75" x2="26" y2="2" width="0.3048" layer="1"/>
-<wire x1="26" y1="2" x2="26" y2="2.5" width="0.3048" layer="1"/>
-</signal>
-<signal name="N$12">
-<contactref element="LED2" pad="A"/>
-<contactref element="R4" pad="1"/>
-<wire x1="30" y1="1.75" x2="31.75" y2="1.75" width="0.3048" layer="1"/>
-<wire x1="31.75" y1="1.75" x2="32" y2="2" width="0.3048" layer="1"/>
-<wire x1="32" y1="2" x2="32" y2="2.5" width="0.3048" layer="1"/>
-</signal>
-<signal name="N$14">
-<contactref element="LED3" pad="A"/>
-<contactref element="R5" pad="1"/>
-<wire x1="36" y1="1.75" x2="37.75" y2="1.75" width="0.3048" layer="1"/>
-<wire x1="37.75" y1="1.75" x2="38" y2="2" width="0.3048" layer="1"/>
-<wire x1="38" y1="2" x2="38" y2="2.5" width="0.3048" layer="1"/>
-</signal>
-<signal name="N$15">
-<contactref element="LED4" pad="A"/>
-<contactref element="R6" pad="1"/>
-<wire x1="18" y1="1.75" x2="19.75" y2="1.75" width="0.3048" layer="1"/>
-<wire x1="19.75" y1="1.75" x2="20" y2="2" width="0.3048" layer="1"/>
-<wire x1="20" y1="2" x2="20" y2="2.5" width="0.3048" layer="1"/>
 </signal>
 <signal name="N$18">
@@
 <via x="5" y="5" extent="1-16" drill="3.2" diameter="6"/>
 </signal>
+<signal name="N$12">
+<contactref element="R3" pad="1"/>
+<contactref element="LED1" pad="C"/>
+<wire x1="26" y1="2.5" x2="25.25" y2="1.75" width="0.3048" layer="1"/>
+<wire x1="25.25" y1="1.75" x2="24" y2="1.75" width="0.3048" layer="1"/>
+</signal>
+<signal name="N$13">
+<contactref element="R4" pad="1"/>
+<contactref element="LED2" pad="C"/>
+<wire x1="32" y1="2.5" x2="31.25" y2="1.75" width="0.3048" layer="1"/>
+<wire x1="31.25" y1="1.75" x2="30" y2="1.75" width="0.3048" layer="1"/>
+</signal>
+<signal name="N$14">
+<contactref element="R5" pad="1"/>
+<contactref element="LED3" pad="C"/>
+<wire x1="38" y1="2.5" x2="37.25" y2="1.75" width="0.3048" layer="1"/>
+<wire x1="37.25" y1="1.75" x2="36" y2="1.75" width="0.3048" layer="1"/>
+</signal>
+<signal name="N$15">
+<contactref element="R6" pad="1"/>
+<contactref element="LED4" pad="C"/>
+<wire x1="20" y1="2.5" x2="19.25" y2="1.75" width="0.3048" layer="1"/>
+<wire x1="19.25" y1="1.75" x2="18" y2="1.75" width="0.3048" layer="1"/>
+</signal>
 </signals>
